Commit message: second commit

File: examen_description/urdf/scara_basic_position_controller.xacro (robot description, xacro)
@@ -1,18 +1,19 @@
 <?xml version="1.0" encoding="utf-8"?>
-<robot name="robot_scara" xmlns:xacros="http://ros/wiki/xacro" >
-    <gazebo>
-        <plugin name="joint-state_publisher_controller" filename="libgazebo_ros_joint_state_publisher.so">
-        <!--update rate Hz-->
-            <update_rate>10</update_rate>
-            <joint_name>link_1_joint</joint_name>
-            <joint_name>link_2_joint</joint_name>
-            <joint_name>link_3_joint</joint_name>
-        </plugin>
-    </gazebo>
-    <gazebo>
-        <plugin name="joint_pose_trajectory_controller" filename="libgazebo_ros_joint_pose_trajectory.so">
-        <!--update rate Hz-->
-            <update_rate>2</update_rate>
-        </plugin>
-    </gazebo>
+<robot name="robot_scara" xmlns:xacro="http://ros.org/wiki/xacro">
+	<gazebo>
+		<plugin name="joint_state_publisher_controller" filename="libgazebo_ros_joint_state_publisher.so">
+			<!-- Update rate Hz -->
+			<update_rate>10</update_rate>
+			<joint_name>link_1_joint</joint_name>
+			<joint_name>link_2_joint</joint_name>
+			<joint_name>link_3_joint</joint_name>
+			<joint_name>link_P_joint</joint_name>
+		</plugin>
+	</gazebo>
+	<gazebo>
+		<plugin name="joint_pose_trajectory_controller" filename="libgazebo_ros_joint_pose_trajectory.so">
+			<!--update rate Hz-->
+			<update_rate>2</update_rate>
+		</plugin>
+	</gazebo>
 </robot>

File: examen_description/urdf/scara_gz_propierties.xacro (robot description, xacro)
@@ -1,15 +1,15 @@
 <?xml version="1.0" encoding="utf-8"?>
-<robot name="robot_scara" xmlns:xacros="http://ros/wiki/xacro" >
-    <gazebo reference="base_link">
-        <material> gazebo/Grey</material>
-    </gazebo>
-    <gazebo reference="link_1">
-        <material> gazebo/Red</material>
-    </gazebo>
-    <gazebo reference="link_2">
-        <material> gazebo/Green</material>
-    </gazebo>
-    <gazebo reference="link_3">
-        <material> gazebo/Blue</material>
-    </gazebo>
+<robot name="robot_scara" xmlns:xacro="http://ros.org/wiki/xacro">
+	<gazebo reference="base_link">
+		<material>Gazebo/Grey</material>
+	</gazebo>
+	<gazebo reference="link_1">
+		<material>Gazebo/Red</material>
+	</gazebo>
+	<gazebo reference="link_2">
+		<material>Gazebo/Green</material>
+	</gazebo>
+	<gazebo reference="link_3">
+		<material>Gazebo/Blue</material>
+	</gazebo>
 </robot>
