Commit message: second commit

File: examen_description/urdf/scara.urdf (robot description, URDF)
Before this commit: robot robot_scara, 6 links, 5 joints
Links:
- removed link P
- removed link world
Joints:
- removed joint link_P_joint
- removed joint world_joint

File: examen_description/urdf/scara_basic_position_controller.xacro (robot description, xacro)
@@ -1,19 +1,17 @@
 <?xml version="1.0" encoding="utf-8"?>
-<robot name="robot_scara" xmlns:xacro="http://ros.org/wiki/xacro">
-	<gazebo>
-		<plugin name="joint_state_publisher_controller" filename="libgazebo_ros_joint_state_publisher.so">
-			<!-- Update rate Hz -->
-			<update_rate>10</update_rate>
-			<joint_name>link_1_joint</joint_name>
-			<joint_name>link_2_joint</joint_name>
-			<joint_name>link_3_joint</joint_name>
-			<joint_name>link_P_joint</joint_name>
-		</plugin>
-	</gazebo>
-	<gazebo>
-		<plugin name="joint_pose_trajectory_controller" filename="libgazebo_ros_joint_pose_trajectory.so">
-			<!--update rate Hz-->
-			<update_rate>2</update_rate>
-		</plugin>
-	</gazebo>
+<robot name="robot_scara" xmlns:xacro="http://ros.org/wiki/xacro" >
+    <gazebo>
+        <plugin name="joint-state_publisher_controller" filename="libgazebo_ros_joint_state_publisher.so">
+            <!--update rate Hz-->
+            <update_rate>10</update_rate>
+            <joint_name>link_1_joint</joint_name>
+            <joint_name>link_2_joint</joint_name>
+            <joint_name>link_3_joint</joint_name>
+        </plugin>
+    </gazebo>
+    <gazebo>
+        <plugin name="joint_pose_trajectory_controller" filename="libgazebo_ros_joint_pose_trajectory.so">
+            <update_rate>2</update_rate>
+        </plugin>
+    </gazebo>
 </robot>

File: examen_description/urdf/scara_position_controller.xacro (robot description, xacro)
@@ -4,4 +4,4 @@
     <xacro:include filename="$(find ${package_name})/urdf/scara_urdf.xacro"/>
     <xacro:include filename="$(find ${package_name})/urdf/scara_gz_properties.xacro"/>
-    <xacro:include filename="$(find ${package_name})/urdf/scara_basic_position_controller.xacro"/>
+    <xacro:include filename="$(find ${package_name})/urdf/position_controller.xacro"/>
 </robot>

File: examen_description/urdf/scara_trajectory_controller.xacro (robot description, xacro)
@@ -4,4 +4,4 @@
     <xacro:include filename="$(find ${package_name})/urdf/scara_urdf.xacro"/>
     <xacro:include filename="$(find ${package_name})/urdf/scara_gz_properties.xacro"/>
-    <xacro:include filename="$(find ${package_name})/urdf/scara_basic_position_controller.xacro"/>
+    <xacro:include filename="$(find ${package_name})/urdf/trajectory_controller.xacro"/>
 </robot>
