Commit message: Exam upload

File: examen_description/urdf/Propuesta2_gz_properties.xacro (robot description, xacro)
@@ -1,15 +1,18 @@
 <?xml version="1.0" encoding="utf-8"?>
 <!--Aqui comienza el robot-->
-<robot name="robot_scara" xmlns:xacro="http://ros.org/wiki/xacro" >
+<robot name="Propuesta2" xmlns:xacro="http://ros.org/wiki/xacro" >
     <gazebo reference="base_link">
         <material>Gazebo/Grey</material>
     </gazebo>
-    <gazebo reference="link_1">
+    <gazebo reference="link_11">
         <material>Gazebo/Red</material>
     </gazebo>
-    <gazebo reference="link_2">
+    <gazebo reference="link_21">
         <material>Gazebo/Blue</material>
     </gazebo>
-    <gazebo reference="link_3">
+    <gazebo reference="link_31">
+        <material>Gazebo/Green</material>
+    </gazebo>
+    <gazebo reference="link_41">
         <material>Gazebo/Green</material>
     </gazebo>

File: examen_description/urdf/Propuesta2_trajectory_controller.xacro (robot description, xacro)
@@ -2,6 +2,6 @@
 <robot name="robot_scara" xmlns:xacro="http://ros.org/wiki/xacro" >
     <xacro:property name="package_name" value="examen_description"/>
-    <xacro:include filename="$(find ${package_name})/urdf/scara_urdf.xacro"/>
-    <xacro:include filename="$(find ${package_name})/urdf/scara_gz_properties.xacro"/>
+    <xacro:include filename="$(find ${package_name})/urdf/Propuesta2_urdf.xacro"/>
+    <xacro:include filename="$(find ${package_name})/urdf/Propuesta2_gz_properties.xacro"/>
     <xacro:include filename="$(find ${package_name})/urdf/trajectory_controller.xacro"/>
 </robot>

File: examen_description/urdf/position_controller.xacro (robot description, xacro)
@@ -1,10 +1,10 @@
 <?xml version="1.0" encoding="utf-8"?>
 <!--Aqui comienza el robot-->
-<robot name="robot_scara" xmlns:xacro="http://ros.org/wiki/xacro" >
+<robot name="Propuesta2" xmlns:xacro="http://ros.org/wiki/xacro" >
     <ros2_control name="GazeboSystem" type="system">
         <hardware>
             <plugin>gazebo_ros2_control/GazeboSystem</plugin>
         </hardware>
-        <joint name="link_1_joint">
+        <joint name="base_link_to_link_1">
             <command_interface name="position"/>
             <state_interface name="position"/>
@@ -12,5 +12,5 @@
             <state_interface name="effort"/>
         </joint>
-        <joint name="link_2_joint">
+        <joint name="link_1_to_link_2">
             <command_interface name="position"/>
             <state_interface name="position"/>
@@ -18,5 +18,11 @@
             <state_interface name="effort"/>
         </joint>
-        <joint name="link_3_joint">
+        <joint name="link_2_to_link_3">
+            <command_interface name="position"/>
+            <state_interface name="position"/>
+            <state_interface name="velocity"/>
+            <state_interface name="effort"/>
+        </joint>
+        <joint name="link_3_to_link_4">
             <command_interface name="position"/>
             <state_interface name="position"/>
@@ -28,5 +34,5 @@
     <gazebo>
         <plugin filename="libgazebo_ros2_control.so" name="gazebo_ros2_control" >
-            <parameters>$(find ${package_name})/config/scara_position_controller.yaml</parameters>
+            <parameters>$(find ${package_name})/config/Propuesta2_position_controller.yaml</parameters>
         </plugin>
     </gazebo>

File: examen_description/urdf/trajectory_controller.xacro (robot description, xacro)
@@ -1,10 +1,10 @@
 <?xml version="1.0" encoding="utf-8"?>
 <!--Aqui comienza el robot-->
-<robot name="robot_scara" xmlns:xacro="http://ros.org/wiki/xacro" >
+<robot name="Propuesta" xmlns:xacro="http://ros.org/wiki/xacro" >
     <ros2_control name="GazeboSystem" type="system">
         <hardware>
             <plugin>gazebo_ros2_control/GazeboSystem</plugin>
         </hardware>
-        <joint name="link_1_joint">
+        <joint name="base_link_to_link_1">
             <command_interface name="position"/>
             <state_interface name="position"/>
@@ -12,5 +12,5 @@
             <state_interface name="effort"/>
         </joint>
-        <joint name="link_2_joint">
+        <joint name="link_1_to_link_2">
             <command_interface name="position"/>
             <state_interface name="position"/>
@@ -18,5 +18,11 @@
             <state_interface name="effort"/>
         </joint>
-        <joint name="link_3_joint">
+        <joint name="link_2_to_link_3">
+            <command_interface name="position"/>
+            <state_interface name="position"/>
+            <state_interface name="velocity"/>
+            <state_interface name="effort"/>
+        </joint>
+        <joint name="link_3_to_link_4">
             <command_interface name="position"/>
             <state_interface name="position"/>
@@ -30,5 +36,5 @@
             <robot_param>robot_description</robot_param>
             <robot_param_node>robot_state_publisher</robot_param_node>
-            <parameters>$(find ${package_name})/config/scara_trajectory_controller.yaml</parameters>
+            <parameters>$(find ${package_name})/config/Propuesta2_trajectory_controller.yaml</parameters>
         </plugin>
     </gazebo>
